File: kicad/kicad.kicad_pcb (KiCad board)
At the start: 2 copper layers, 315 x 123 mm, 54 parts, among them J1 Conn_01x16_Pin, K0 !,,,,,,1, K1 ",,,,,,2, K10 *,,,,,,:, K11 =,,,,,,-, K12 Break, K13 Up, K14 Q, K15 W, K16 E, K17 R, K18 T, K19 Y, K2 #,,,,,,3, K20 U, K21 I, K22 O, K23 P, K24 @, K25 Left, K26 Right, K27 Down, K28 A, K29 S, K3 $,,,,,,4, K30 D, K31 F, K32 G, K33 H, K34 J, K35 K, K36 L, K37 +,,,,,,;, K38 ENTER, K39 CLEAR, K4 %,,,,,,5, K40 SHIFT, K41 Z, K42 X, K43 C, K44 V, K45 B, K46 N, K47 M, K48 <,,,,,,,, K49 >,,,,,,., K5 &,,,,,,6, K50 ?,,,,,,/, K51 SHIFT, K52 Blank, K6 ',,,,,,7, K7 (,,,,,,8, K8 ),,,,,,9, K9 0

Commit message: Pin labels
Other:
- board text added: "Col 1"
- board text added: "Col 2"
- board text added: "Col 3"
- board text added: "Col 4"
- board text added: "Col 5"
- board text added: "Col 6"
- board text added: "Col 7"
- board text added: "Col 8"
- board text added: "KEY"
- board text added: "Row 1"
- board text added: "Row 2"
- board text added: "Row 3"
- board text added: "Row 4"
- board text added: "Row 5"
- board text added: "Row 6"
- board text added: "Row 7"
Changed lines of the file:
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@@
 		(layer "Edge.Cuts")
+	)
+	(gr_text "Col 4"
+		(at 236.855 83.82 -90)
+		(layer "B.SilkS")
+		(effects
+			(font
+				(size 1 1)
+				(thickness 0.15)
+			)
+			(justify left bottom mirror)
+		)
+	)
+	(gr_text "Col 3"
+		(at 234.315 83.82 -90)
+		(layer "B.SilkS")
+		(effects
+			(font
+				(size 1 1)
+				(thickness 0.15)
+			)
+			(justify left bottom mirror)
+		)
+	)
+	(gr_text "Col 7"
+		(at 244.475 83.82 -90)
+		(layer "B.SilkS")
+		(effects
+			(font
+				(size 1 1)
+				(thickness 0.15)
+			)
+			(justify left bottom mirror)
+		)
+	)
+	(gr_text "Col 6"
+		(at 241.935 83.82 -90)
+		(layer "B.SilkS")
+		(effects
+			(font
+				(size 1 1)
+				(thickness 0.15)
+			)
+			(justify left bottom mirror)
+		)
+	)
+	(gr_text "Row 4"
+		(at 219.075 83.82 270)
+		(layer "B.SilkS")
+		(effects
+			(font
+				(size 1 1)
+				(thickness 0.15)
+			)
+			(justify left bottom mirror)
+		)
+	)
+	(gr_text "Col 2"
+		(at 231.775 83.82 -90)
+		(layer "B.SilkS")
+		(effects
+			(font
+				(size 1 1)
+				(thickness 0.15)
+			)
+			(justify left bottom mirror)
+		)
+	)
+	(gr_text "Row 5"
+		(at 221.615 83.82 -90)
+		(layer "B.SilkS")
+		(effects
+			(font
+				(size 1 1)
+				(thickness 0.15)
+			)
+			(justify left bottom mirror)
+		)
+	)
+	(gr_text "Col 8"
+		(at 247.015 83.82 -90)
+		(layer "B.SilkS")
+		(effects
+			(font
+				(size 1 1)
+				(thickness 0.15)
+			)
+			(justify left bottom mirror)
+		)
+	)
+	(gr_text "Row 3"
+		(at 216.535 83.82 -90)
+		(layer "B.SilkS")
+		(effects
+			(font
+				(size 1 1)
+				(thickness 0.15)
+			)
+			(justify left bottom mirror)
+		)
+	)
+	(gr_text "KEY"
+		(at 213.995 83.82 -90)
+		(layer "B.SilkS")
+		(effects
+			(font
+				(size 1 1)
+				(thickness 0.15)
+			)
+			(justify left bottom mirror)
+		)
+	)
+	(gr_text "Col 1"
+		(at 229.235 83.82 -90)
+		(layer "B.SilkS")
+		(effects
+			(font
+				(size 1 1)
+				(thickness 0.15)
+			)
+			(justify left bottom mirror)
+		)
+	)
+	(gr_text "Row 2"
+		(at 211.455 83.82 -90)
+		(layer "B.SilkS")
+		(effects
+			(font
+				(size 1 1)
+				(thickness 0.15)
+			)
+			(justify left bottom mirror)
+		)
+	)
+	(gr_text "Row 7"
+		(at 226.695 83.82 -90)
+		(layer "B.SilkS")
+		(effects
+			(font
+				(size 1 1)
+				(thickness 0.15)
+			)
+			(justify left bottom mirror)
+		)
+	)
+	(gr_text "Col 5"
+		(at 239.395 83.82 -90)
+		(layer "B.SilkS")
+		(effects
+			(font
+				(size 1 1)
+				(thickness 0.15)
+			)
+			(justify left bottom mirror)
+		)
+	)
+	(gr_text "Row 1"
+		(at 208.915 83.82 270)
+		(layer "B.SilkS")
+		(effects
+			(font
+				(size 1 1)
+				(thickness 0.15)
+			)
+			(justify left bottom mirror)
+		)
+	)
+	(gr_text "Row 6"
+		(at 224.155 83.82 -90)
+		(layer "B.SilkS")
+		(effects
+			(font
+				(size 1 1)
+				(thickness 0.15)
+			)
+			(justify left bottom mirror)
+		)
 	)
 	(gr_text "coco keyboard insert v1\nleadedsolder.com 2024"
